File: Schematics/CapstoneSchematic.sch (KiCad schematic (older format))
At the start: 19 parts

Commit message: Did main pcb
Parts:
- removed 47kOhm: R, symbol Device:R
- removed D_GREEN, D_RED: LED, symbol Device:LED
- removed R1, R2: 220, symbol Device:R
- removed R?: R_PHOTO, symbol Device:R_PHOTO
- removed UReg?: LinearRegulatorPCB, symbol CapstoneSchematic-cache:CapstoneSchematic-cache_CapstoneSchematic-cache_Capston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
- added J2: VoltageIn, TerminalBlock_MetzConnect:TerminalBlock_MetzConnect_Type094_RT03502HBLU_1x02_P5.00mm_Horizontal, symbol Connector:Screw_Terminal_01x02
- added LED_GREEN1, LED_RED1: 200, TerminalBlock_MetzConnect:TerminalBlock_MetzConnect_Type094_RT03502HBLU_1x02_P5.00mm_Horizontal, symbol CapstoneSchematic:LEDModule
- added LR1: Linear_Regulator, Capstone_PCB_Lib:Linear Regulator, symbol CapstoneSchematic:Linear_Regulator
- added PR1: PhotoResistor, TerminalBlock_MetzConnect:TerminalBlock_MetzConnect_Type094_RT03503HBLU_1x03_P5.00mm_Horizontal, symbol CapstoneSchematic:PhotoResistor
- added U6: LaserSensor, TerminalBlock_MetzConnect:TerminalBlock_MetzConnect_Type094_RT03503HBLU_1x03_P5.00mm_Horizontal, symbol CapstoneSchematic:LaserSensor
- J1: renamed from J?; footprint (none) -> Connector_PinSocket_2.54mm:PinSocket_1x04_P2.54mm_Vertical; symbol CapstoneSchematic-rescue:ArduinoRGBShield -> CapstoneSchematic:ArduinoRGBShield
- RM1: renamed from U?; footprint (none) -> Capstone_PCB_Lib:2 Channels Relay; symbol CapstoneSchematic-rescue:2RelayModule-CapstoneLib -> CapstoneSchematic:2RelayModule
- SAS1: renamed from U?; footprint (none) -> TerminalBlock_MetzConnect:TerminalBlock_MetzConnect_Type094_RT03503HBLU_1x03_P5.00mm_Horizontal; symbol CapstoneSchematic-rescue:SnapActionSwitch-CapstoneLib -> CapstoneSchematic:SnapActionSwitch
- SAS2: renamed from U?; footprint (none) -> TerminalBlock_MetzConnect:TerminalBlock_MetzConnect_Type094_RT03502HBLU_1x02_P5.00mm_Horizontal; symbol CapstoneSchematic-rescue:SnapActionSwitch-CapstoneLib -> CapstoneSchematic:SnapActionSwitch
- T1: renamed from U?; value MCP9700AT-ELT -> Temp Sensor; footprint Package_TO_SOT_SMD:SOT-353_SC-70-5 -> TerminalBlock_MetzConnect:TerminalBlock_MetzConnect_Type094_RT03503HBLU_1x03_P5.00mm_Horizontal
- U1: renamed from U?; symbol CapstoneSchematic-rescue:LinearActuator-CapstoneLib -> CapstoneSchematic:LinearActuator
- U7: renamed from U?; symbol CapstoneSchematic-rescue:CMP12-CapstoneLib -> CapstoneSchematic:CMP12
- ULoRa1: renamed from ULoRa?; footprint (none) -> Connector_PinSocket_2.54mm:PinSocket_1x06_P2.54mm_Horizontal; symbol CapstoneSchematic-rescue:LoRa-CapstoneLib -> CapstoneSchematic:LoRa
- gave numbers to parts that had none: 3
- renumbered 2A to 2A1
Connections:
- net labels added: 0
- net labels removed: -12V
- wire segments 76 -> 77
