File: Schematics/CapstoneSchematic.sch (KiCad schematic (older format))
At the start: 20 parts, among them J1 ArduinoRGBShield, J2 VoltageIn, T1 Temp Sensor, U1 LinearActuator, U6 LaserSensor, U7 CMP12-CapstoneLib

Commit message: finished pcb
Parts:
- removed U1: LinearActuator, symbol CapstoneSchematic:LinearActuator
- added LA1: LinearActuator, symbol CapstoneSchematic:LinearActuator
- SAS1: footprint TerminalBlock_MetzConnect:TerminalBlock_MetzConnect_Type094_RT03503HBLU_1x03_P5.00mm_Horizontal -> TerminalBlock_MetzConnect:TerminalBlock_MetzConnect_Type094_RT03502HBLU_1x02_P5.00mm_Horizontal
- SAS2: footprint TerminalBlock_MetzConnect:TerminalBlock_MetzConnect_Type094_RT03502HBLU_1x02_P5.00mm_Horizontal -> TerminalBlock_MetzConnect:TerminalBlock_MetzConnect_Type094_RT03503HBLU_1x03_P5.00mm_Horizontal
Connections:
- net +12V: now also 2A1.2, J2.1 (Pin_1), RM1.9 (COMM); no longer J2.2 (Pin_2)
- net 0: now also J2.2 (Pin_2); no longer J2.1 (Pin_1)
- net at A1.11 (A2): now also PR1.2
- net LoRa3: now reaches ULoRa1.3 (RXD)
- net LoRa3: now also A1.16 (D1/TX); no longer A1.15 (D0/RX)
- net LoRa4: now reaches ULoRa1.4 (TXD)
- net LoRa4: now also A1.15 (D0/RX); no longer A1.16 (D1/TX)
- net SAS_Int1: now reaches A1.17 (D2), SAS1.4 (NO_T1)
- net SAS_Int2: now reaches A1.18 (D3), SAS2.4 (NO_T1)
- net at A1.19 (D4): now also U6.3 (DAT); no longer ULoRa1.2 (NRST)
- net at MPS1.3 (Dout): now also A1.27 (D12); no longer A1.20 (D5)
- net at MPS2.3 (Dout): now also A1.28 (D13); no longer A1.21 (D6)
- net LED_G: now reaches A1.22 (D7)
- net LED_G: now also LED_GREEN1.2
- net at A1.23 (D8): no longer LED_GREEN1.2
- net IN1: now reaches A1.24 (D9)
- net IN1: now also RM1.2 (In1); no longer LED_RED1.2
- net IN2: now reaches A1.25 (D10)
- net IN2: now also RM1.3 (In2)
- net at A1.26 (D11): no longer U6.3 (DAT)
- net at A1.9 (A0): no longer PR1.2
- net at RM1.6 (COMM): now also SAS2.2 (COM_T2); no longer SAS1.2 (COM_T2)
- net at 2A1.1: now also LA1.2 (Vpos); no longer RM1.9 (COMM)
- new net: LA1.1 (VNeg), SAS1.2 (COM_T2)
- new net LED_R: A1.21 (D6), LED_RED1.2
- new net LoRa2: A1.20 (D5), ULoRa1.2 (NRST)
Other:
- moved on the sheet: 2A1, A1, BT1, J1, J2, LED_GREEN1, LED_RED1, LR1, PR1, RM1, SAS1, SAS2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

Commit message: Jacob and Nathan working on the project
Connections:
- net +12V: no longer 2A1.2, RM1.9 (COMM)
- new net: 2A1.2, RM1.9 (COMM)
Other:
- note added: "Notes:\nThere was an accidental junction on the Common and 12V for the Relays, need to fix\n\nInterrupts need rewiring: https://www.instructables.com/id/Arduino-Interrupts/\n-THe COMM goes to GND for 5V line\n\nLinear Reg,put pin names on silkscreen\n\nLED_G should just go to 5V line and not be connected to arduino.\n\nMake AREF Accessible"
Changed lines of the file:
@@
 $EndComp
-Wire Wire Line
-	1950 3900 1950 3800
-Wire Wire Line
-	1950 3050 2400 3050
-Connection ~ 1950 3800
-Wire Wire Line
-	1950 3800 1950 3050
 Wire Wire Line
 	1950 4250 2750 4250
@@
 Wire Wire Line
 	6650 4050 6650 5750
+Wire Wire Line
+	2350 3050 2350 3900
+Wire Wire Line
+	2350 3050 2400 3050
+Wire Wire Line
+	1950 3900 2350 3900
+Text Notes 1000 5800 0    50   ~ 0
+Notes:\nThere was an accidental junction on the Common and 12V for the Relays, need to fix\n\nInterrupts need rewiring: https://www.instructables.com/id/Arduino-Interrupts/\n-THe COMM goes to GND for 5V line\n\nLinear Reg,put pin names on silkscreen\n\nLED_G should just go to 5V line and not be connected to arduino.\n\nMake AREF Accessible
 Wire Bus Line
 	695  4050 695  4885
